File: qi_experiments_pcb/qi_experiments_pcb.kicad_pcb (KiCad board)
At the start: 4 copper layers, 71 x 34.5 mm, 70 parts, among them J1 Conn_01x03, J2 USB_C_Receptacle_USB2.0, J3 Conn_01x02, J4 Conn_01x02, Q1 2N7002, Q2 2N7002, Q3 2N7002, U2 SPX3819M5-L-3-3, U4 AP62200Z6, U5 CH340N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

Commit message: curent sensing amp polarity swap
Parts:
- R12: value R -> 470
- R5: value R -> 1k
- turned R3 to 180 degrees
Connections:
- R16 pad 1: Net-(C6-Pad2) -> GND
- R17 pad 1: GND -> Net-(C6-Pad2)
Routing:
- net Net-(C6-Pad2): track 32.0 -> 29.3 mm
Other:
- board text added: "Qi_experiments_v1.1"
- board text added: "v1.1"
- board text removed: "Qi_experiments_v1.0"
- board text removed: "v1.0"
